File: cableTesterUsbTypeC.kicad_sch (KiCad schematic)
At the start: 53 parts, among them J1 USB_C_Receptacle, J3 USB_C_Receptacle

Commit message: Add LCSC BOM file to the v0.1 archive
Parts:
- BT1: LCSC (none) -> C70377; MPN (none) -> CR2032-BS-6-1
- D1, D10, D11, D12, D13, D14, D15, D16, D17, D18, D19, D2, D20, D21, D22, D23, D24, D25, D3, D4, D5, D6, D7, D8, D9: LCSC (none) -> C965815; MPN (none) -> XL-2012UGC
- J1, J3: LCSC (none) -> C2919640; MPN (none) -> KH-TYPE-C-JB0.8-24P
- R1, R10, R11, R12, R13, R14, R15, R16, R17, R18, R19, R2, R20, R21, R22, R23, R24, R25, R3, R4, R5, R6, R7, R8, R9: LCSC (none) -> C2907294; MPN (none) -> FRC0805J101 TS
